File: pi_day_2025.brd (EAGLE design)
At the start: 50.8 x 25.4 mm, 66 parts, among them IC1 W25Q64JVXGIQ, IC2 ZMOD4510AI1R, J1 SM06B-GHS-TB(LF)(SN), J3 TF-123-ARP9HXX, J4 SM03B-SRSS-TB(LF)(SN), Q2 BSS138, U1 APS6404L-3SQR-ZR, U2 RP2350A, U3 MIC5504-3.3YM5_TR, U4 BME690, Y1 12MHz

Commit message: design file check-in
Parts:
- removed C16, C19, C2, C22, C23, C24, C25, C26: 0.1uF, SparkFun-Capacitors:0402
- removed IC2: ZMOD4510AI1R, ZMOD4510AI1R:ZMOD4510AI1R
- removed J1: SM06B-GHS-TB(LF)(SN), SM06B-GHS-TB_LF__SN_:JST_SM06B-GHS-TB(LF)(SN)
- removed J2: (no value), SparkFun-Connectors:1X04_1MM_RA
- removed J3: TF-123-ARP9HXX, xunpu_tf123:MICROSDCARD
- removed LED1: WS2812B-2020, WS2812B-2020:WS2812B-2020
- removed R9: 10K, SparkFun-Resistors:0402@1
- removed U4: BME690, BME690:IC_BME688
- D2: value BLUE -> SK6812-EJ; device APHHS1005LQBC_D-V:LED_APHHS1005LQBC/D-V -> SK6812-E:LED_SK6812-E
- moved D2 49.4 mm to (-9.91, -33.0), turned to 0 degrees
Connections:
- removed net BME690_CSB: U2.33, U4.2
- removed net BME690_SCK: U2.34, U4.4
- removed net BME690_SDI: U2.35, U4.3
- removed net BME690_SDO: U2.32, U4.5
- removed net CMD: J3.P3, U2.19
- removed net DAT0: J3.P7, U2.16
- removed net DAT1: J3.P8, U2.15
- removed net DAT2: J3.P1, U2.14
- removed net DAT3: J3.P2, U2.17
- removed net INT_ZMOD4510: IC2.3, U2.28
- removed net RES_ZMOD4510: IC2.11, R9.1, U2.29
- removed net SD_CLK: J3.P5, U2.18
- removed net SWITCH: J3.G1, U2.13
- new net VDD: D2.1
- net 3.3V: no longer C16.1, C19.1, C22.1, C23.1, C24.2, C25.2, C26.1, IC2.10, IC2.12, IC2.5, J2.2, J3.P4, LED1.4, R9.2, U4.6, U4.8
- net GND: now also D2.3; no longer C16.2, C19.2, C2.2, C22.2, C23.2, C24.1, C25.1, C26.2, D2.1, IC2.6, IC2.7, IC2.9, J1.2, J1.5, J1.S1, J1.S2, J2.1, J3.P$1, J3.P$2, J3.P$3, J3.P$4, J3.P6, LED1.2, U4.1, U4.7
- net N$4: no longer D2.2
- net NEOPIXEL: no longer LED1.3
- net SCL: no longer IC2.1, J1.4, J2.4
- net SDA: no longer IC2.2, J1.3, J2.3
- net V_USB: no longer C2.1, J1.1
Routing:
- net INT_ZMOD4510: track 37.9 -> 0.00 mm, vias 2 -> 0
- net BME690_SDI: track 34.2 -> 0.00 mm, vias 2 -> 0
- net RES_ZMOD4510: track 33.5 -> 0.00 mm, vias 2 -> 0
- net BME690_SCK: track 31.8 -> 0.00 mm, vias 2 -> 0
- net BME690_SDO: track 31.6 -> 0.00 mm
- net BME690_CSB: track 31.3 -> 0.00 mm, vias 2 -> 0
- net 3.3V: track 80.5 -> 55.8 mm, vias 25 -> 16
- net DAT2: track 21.2 -> 0.00 mm, vias 2 -> 0
- net DAT3: track 19.3 -> 0.00 mm, vias 2 -> 0
- net CMD: track 19.2 -> 0.00 mm
- net SWITCH: track 17.9 -> 0.00 mm, vias 2 -> 0
- net SD_CLK: track 17.1 -> 0.00 mm
- net DAT0: track 13.9 -> 0.00 mm
- net DAT1: track 13.7 -> 0.00 mm
- net SDA: track 62.8 -> 56.6 mm
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
Commit message: Updates to design
Parts:
- removed C14, C15: 10uF, OPL_Capacitor:C0402
- removed U3: MIC5504-3.3YM5_TR, MIC5504-3.3YM5_TR:SOT95P280X145-5N
- added C10, C11, C2, C3, C4, C5, C6, C7, C8, C9: 0.1uF, SparkFun-Capacitors:0402
- added D10, D3, D4, D5, D6, D7, D8, D9: SK6812-EJ, SK6812-E:LED_SK6812-E
- added U4: LTC4088EDE#PBF, LTC4088EDE_PBF:SON50P300X400X80-15N
- D1: value 1N4148 -> SK6812-EJ; device SparkFun-DiscreteSemi:SOD-323 -> SK6812-E:LED_SK6812-E
- moved D1 69.0 mm to (-14.7, -42.9)
- moved D2 23.9 mm to (-14.7, -56.4)
Connections:
- removed net VDD: D2.1
- new net BAT: U4.9
- new net SW: U4.12
- new net VBUS: U4.11
- new net VOUT: U4.10
- net 3.3V: now also C10.1, C11.1, C2.1, C3.1, C4.1, C5.1, C6.1, C7.1, C8.1, C9.1, D1.1, D10.1, D2.1, D3.1, D4.1, D5.1, D6.1, D7.1, D8.1, D9.1; no longer C15.2, D1.C, U3.5
- net GND: now also C10.2, C11.2, C2.2, C3.2, C4.2, C5.2, C6.2, C7.2, C8.2, C9.2, D1.3, D10.3, D3.3, D4.3, D5.3, D6.3, D7.3, D8.3, D9.3, U4.15; no longer C14.1, C15.1, U3.2
- net N$26: no longer D1.A
- net V_USB: no longer C14.2, U3.1, U3.3
Routing:
- net V_USB: track 63.1 -> 1.68 mm, vias 2 -> 0
- net 3.3V: track 55.8 -> 52.9 mm, vias 16 -> 14
- net N$26: track 3.82 -> 1.64 mm

Commit message: File upload
Parts:
- added C14, C15: 10uF, SparkFun-Capacitors:0805
- added D11: BLUE, SparkFun-LED:LED-0603
- added Q1: Si2333, SparkFun-DiscreteSemi:SOT23-3
- Q2: value BSS138 -> 310mA/60V/1.6Ω
Connections:
- removed net NEOPIXEL: U2.27
- removed net VOUT: U4.10
- net 3.3V: now also C14.1, U4.10, U4.3
- net GND: now also C14.2, C15.2, D11.C, Q1.1
- net N$4: now also D11.A
- net N$9: now also Q1.2; no longer CONN1.A4, CONN1.A9, CONN1.B4, CONN1.B9
- net VBUS: now also CONN1.A4, CONN1.A9, CONN1.B4, CONN1.B9, Q1.3; no longer U4.11
- net V_USB: now also C15.1, U4.11
Routing:
- net NEOPIXEL: track 22.9 -> 0.00 mm, vias 2 -> 0
- net N$9: track 24.2 -> 19.2 mm

Commit message: Check-in
Parts:
- added C16: 0.1uF, SparkFun-Capacitors:0402
- added C19: 0.1uF, SparkFun-Capacitors:0402-TIGHT
- added D12: 1N5819HW-7, 1N5819HW-7:SOD3715X145N
- added J1: (no value), SparkFun-Connectors:JST-2-SMD
- added L3: ASPI-0602S-3R3M-T, ASPI-0602S-3R3M-T:IND_ASPI-0602S-3R3M-T
- added MK1: SPK2611HM7H-1-6, SPK2611HM7H-1-6:MIC_SPK2611HM7H-1-6
- added Q3: Si2333, SparkFun-DiscreteSemi:SOT23-3
- added R10: 2.94K, SparkFun-Resistors:0402
- added R14: 8.2, SparkFun-Resistors:0402
- added R16: 100K, SparkFun-Resistors:0402
- added R17: 100k, SparkFun-Resistors:0603
- added R9: 499, SparkFun-Resistors:0402
- added U3: TPS76318DBVRG4, TPS76318DBVRG4:SOT95P280X145-5N
- added U5: TXS0108EPWRG4, TXS0108EPWRG4:SOP65P640X120-20N
- added U6: LSM6DS3TR-C, LSM6DS3TR-C:LGA-14-2.5X3MM
- R3, R8: value 5.1K -> (none); device SparkFun-Resistors:0402@1 -> SparkFun-Resistors:0402
- R4: device SparkFun-Resistors:0402@1 -> SparkFun-Resistors:0402
- R5: value 10K -> (none); device SparkFun-Resistors:0402@1 -> SparkFun-Resistors:0402
- R6, R7: value 2.2K -> (none); device SparkFun-Resistors:0402@1 -> SparkFun-Resistors:0402
Connections:
- removed net BAT: U4.9
- removed net SW: U4.12
- new net 1.8V: MK1.1
- new net LSM6_INT1: U6.4
- new net LSM6_INT2: U6.9
- new net N$10: J1.2, Q3.3, U4.9
- new net N$14: R9.2, U4.5, U4.6
- new net N$15: R10.2, R14.2, U4.2
- new net N$16: C16.1, R14.1
- new net N$17: R16.1, R17.1, U4.1
- new net N$6: L3.2, U4.12
- new net N$8: Q3.1, U4.8
- new net NPXL_1_IN: D1.4, U2.13
- new net NPXL_1_OUT: D1.2, D2.4
- new net NPXL_2_OUT: D2.2, D3.4
- new net NPXL_3_OUT: D3.2, D4.4
- new net NPXL_4_OUT: D4.2, D5.4
- new net NPXL_5_OUT: D5.2, D6.4
- new net NPXL_6_OUT: D6.2, D7.4
- new net NPXL_7_OUT: D7.2, D8.4
- new net NPXL_8_OUT: D8.2, D9.4
- new net NPXL_9_OUT: D10.4, D9.2
- new net VCCA: U5.2
- new net VCCB: U5.19
- net 3.3V: now also C19.1, D12.C, L3.1, Q3.2, U6.1, U6.12, U6.5, U6.8
- net GND: now also C16.2, C19.2, J1.1, MK1.7, R10.1, R17.2, R9.1, U3.2, U4.13, U4.4, U5.11, U6.2, U6.3, U6.6, U6.7
- net N$26: now also D12.A
- net SCL: now also U6.13
- net SDA: now also U6.14
- net V_USB: now also R16.2, U4.14

Commit message: Check-in
Parts:
- removed L3: ASPI-0602S-3R3M-T, ASPI-0602S-3R3M-T:IND_ASPI-0602S-3R3M-T
- removed Q1, Q3: Si2333, SparkFun-DiscreteSemi:SOT23-3
- added C20: 1.0uF, SparkFun-Capacitors:0402
- added D13, D14, D15: GREEN, SparkFun-LED:LED-0603
- added R18, R19: 220, SparkFun-Resistors:0402-TIGHT
- added R20: 1K, SparkFun-Resistors:0402
- added U7: MCP73833T-AMI/MF, MCP73833T-AMI_MF:SON50P300X300X100-11N
- added U8: TPS2113APWR, TPS2113APWR:SOP65P640X120-8N
- C14, C15: value 10uF -> 0.1uF; device SparkFun-Capacitors:0805 -> SparkFun-Capacitors:0402
- C16: value 0.1uF -> 1.0uF
- L1: value 3.9NH -> 2.2nH; device SparkFun-Coils:0402 -> LQW18AN2N2D10D:INDC1608X100N
- R10: value 2.94K -> 100K
- R14: value 8.2 -> 500
- R16: value 100K -> 220; device SparkFun-Resistors:0402 -> SparkFun-Resistors:0402-TIGHT
- R17: value 100k -> 10k
- R3, R8: value (none) -> 5.1K
- R4: value DNF -> (none)
- R9: value 499 -> 100K
- U4: value LTC4088EDE#PBF -> TPS63001DRCR; device LTC4088EDE_PBF:SON50P300X400X80-15N -> TPS63001DRCR:VREG_V62/16624-01YE
- moved U4 175.5 mm to (-61.0, -204.0)
- moved C15 90.9 mm to (-75.7, -238.3)
- moved C14 81.2 mm to (-67.1, -225.6)
- moved J1 69.7 mm to (-73.4, -226.8)
- moved C16 67.3 mm to (-75.7, -241.6)
- moved R17 57.3 mm to (-75.7, -234.9)
- moved R10 49.4 mm to (-67.1, -218.9)
- moved R14 49.4 mm to (-67.1, -222.2)
- moved R9 49.4 mm to (-67.1, -215.6)
- moved R16 49.2 mm to (-67.1, -228.6)
Connections:
- new net CHARGE_STAT: U2.3, U7.3
- new net N$18: D15.C, U7.4
- new net N$19: R20.2, U7.6
- new net VIN: U8.7
- new net V_BATT: C15.1, C20.1, J1.2, U7.10, U7.9, U8.6
- net 3.3V: no longer C14.1, L3.1, Q3.2, U4.10, U4.3
- net GND: now also C14.1, C16.1, C20.2, R10.2, R14.1, R17.1, R20.1, U4.11, U4.12, U4.14, U4.3, U4.9, U7.11, U7.5, U8.2, U8.5; no longer C14.2, C16.2, Q1.1, R10.1, R17.2, R9.1, U4.4
- net N$10: now also D13.C, U8.1; no longer J1.2, Q3.3, U4.9
- net N$14: now also R17.2, U7.8; no longer R9.2, U4.5, U4.6
- net N$15: now also D14.A, R18.1; no longer R10.2, R14.2, U4.2
- net N$16: now also D14.C, U7.7; no longer C16.1, R14.1
- net N$17: now also D15.A, R19.1; no longer R16.1, R17.1, U4.1
- net N$6: now also R10.1, R9.2, U8.3; no longer L3.2, U4.12
- net N$8: now also R14.2, U8.4; no longer Q3.1, U4.8
- net N$9: now also D13.A, R16.1; no longer C12.1, L1.1, Q1.2
- net VBUS: now also C12.1, L1.1; no longer Q1.3
- net V_USB: now also C14.2, C16.2, R18.2, R19.2, R9.1, U7.1, U7.2, U8.8; no longer C15.1, U4.11, U4.14
Routing:
- net N$9: track 19.2 -> 0.00 mm, vias 2 -> 0
- net VBUS: track 0.00 -> 19.0 mm, vias 0 -> 2

Commit message: Finished power supply design
Parts:
- added C21, C22, C23: 10uF, SparkFun-Capacitors:0402-TIGHT
- added C24: 0.1uF, SparkFun-Capacitors:0402
- added L3: LQH3NPN2R2MJRL, LQH3NPN2R2MJRL:IND_LQH3NPN2R2MJRL
- added R21: 100, SparkFun-Resistors:0402-TIGHT
Connections:
- new net N$20: L3.2, U4.4
- new net N$21: L3.1, U4.2
- new net N$22: C24.1, R21.1, U4.6, U4.7, U4.8
- net 3.3V: now also C21.1, C22.1, U4.1, U4.10
- net GND: now also C21.2, C22.2, C23.2, C24.2
- net VIN: now also C23.1, R21.2, U4.5
Changed lines of the file:
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@@
 <attribute name="VALUE" x="-75.692" y="-260.858" size="0.6096" layer="27" font="vector" ratio="20" align="top-center"/>
+</element>
+<element name="C21" library="SparkFun-Capacitors" library_urn="urn:adsk.eagle:library:510" package="0402-TIGHT" package3d_urn="urn:adsk.eagle:package:41385069/1" value="10uF" x="-75.692" y="-263.144" smashed="yes">
+<attribute name="NAME" x="-75.692" y="-262.582" size="0.6096" layer="25" font="vector" ratio="20" align="bottom-center"/>
+<attribute name="PROD_ID" value="CAP-14848" x="-75.692" y="-263.144" size="1.778" layer="27" display="off"/>
+<attribute name="VALUE" x="-75.692" y="-263.706" size="0.6096" layer="27" font="vector" ratio="20" align="top-center"/>
+</element>
+<element name="C22" library="SparkFun-Capacitors" library_urn="urn:adsk.eagle:library:510" package="0402-TIGHT" package3d_urn="urn:adsk.eagle:package:41385069/1" value="10uF" x="-75.692" y="-266.192" smashed="yes">
+<attribute name="NAME" x="-75.692" y="-265.63" size="0.6096" layer="25" font="vector" ratio="20" align="bottom-center"/>
+<attribute name="PROD_ID" value="CAP-14848" x="-75.692" y="-266.192" size="1.778" layer="27" display="off"/>
+<attribute name="VALUE" x="-75.692" y="-266.754" size="0.6096" layer="27" font="vector" ratio="20" align="top-center"/>
+</element>
+<element name="L3" library="LQH3NPN2R2MJRL" package="IND_LQH3NPN2R2MJRL" value="LQH3NPN2R2MJRL" x="-74.168" y="-271.526" smashed="yes">
+<attribute name="AVAILABILITY" value="In Stock" x="-74.168" y="-271.526" size="1.778" layer="27" display="off"/>
+<attribute name="CHECK_PRICES" value="https://www.snapeda.com/parts/LQH3NPN2R2MJRL/Murata/view-part/?ref=eda" x="-74.168" y="-271.526" size="1.778" layer="27" display="off"/>
+<attribute name="DESCRIPTION" value="                                                      Inductor with Inductance: 2.2uH Tol. +/-20%, Package: 1212 (3030)                                              " x="-74.168" y="-271.526" size="1.778" layer="27" display="off"/>
+<attribute name="MF" value="Murata" x="-74.168" y="-271.526" size="1.778" layer="27" display="off"/>
+<attribute name="MP" value="LQH3NPN2R2MJRL" x="-74.168" y="-271.526" size="1.778" layer="27" display="off"/>
+<attribute name="NAME" x="-76.948" y="-269.526" size="1.27" layer="25"/>
+<attribute name="PACKAGE" value="NONSTANDARD " x="-74.168" y="-271.526" size="1.778" layer="27" display="off"/>
+<attribute name="PRICE" value="None" x="-74.168" y="-271.526" size="1.778" layer="27" display="off"/>
+<attribute name="SNAPEDA_LINK" value="https://www.snapeda.com/parts/LQH3NPN2R2MJRL/Murata/view-part/?ref=snap" x="-74.168" y="-271.526" size="1.778" layer="27" display="off"/>
+<attribute name="VALUE" x="-76.948" y="-273.526" size="1.27" layer="27" align="top-left"/>
+</element>
+<element name="C23" library="SparkFun-Capacitors" library_urn="urn:adsk.eagle:library:510" package="0402-TIGHT" package3d_urn="urn:adsk.eagle:package:41385069/1" value="10uF" x="-75.692" y="-276.86" smashed="yes">
+<attribute name="NAME" x="-75.692" y="-276.298" size="0.6096" layer="25" font="vector" ratio="20" align="bottom-center"/>
+<attribute name="PROD_ID" value="CAP-14848" x="-75.692" y="-276.86" size="1.778" layer="27" display="off"/>
+<attribute name="VALUE" x="-75.692" y="-277.422" size="0.6096" layer="27" font="vector" ratio="20" align="top-center"/>
+</element>
+<element name="R21" library="SparkFun-Resistors" library_urn="urn:adsk.eagle:library:532" package="0402-TIGHT" package3d_urn="urn:adsk.eagle:package:41389023/1" value="100" x="-75.692" y="-279.908" smashed="yes">
+<attribute name="NAME" x="-75.692" y="-279.346" size="0.6096" layer="25" font="vector" ratio="20" align="bottom-center"/>
+<attribute name="PROD_ID" value="RES-14962" x="-75.692" y="-279.908" size="1.778" layer="27" display="off"/>
+<attribute name="VALUE" x="-75.692" y="-280.47" size="0.6096" layer="27" font="vector" ratio="20" align="top-center"/>
+</element>
+<element name="C24" library="SparkFun-Capacitors" library_urn="urn:adsk.eagle:library:510" package="0402" package3d_urn="urn:adsk.eagle:package:41385089/1" override_package3d_urn="urn:adsk.eagle:package:44163386/2" override_package_urn="urn:adsk.eagle:footprint:37389/1" value="0.1uF" x="-75.692" y="-282.956" smashed="yes">
+<attribute name="NAME" x="-75.692" y="-282.194" size="0.6096" layer="25" font="vector" ratio="20" align="bottom-center"/>
+<attribute name="PROD_ID" value="CAP-12416" x="-75.692" y="-282.956" size="1.778" layer="27" display="off"/>
+<attribute name="VALUE" x="-75.692" y="-283.718" size="0.6096" layer="27" font="vector" ratio="20" align="top-center"/>
 </element>
 </elements>
@@
 <contactref element="U4" pad="13"/>
 <contactref element="U4" pad="15"/>
+<contactref element="C21" pad="2"/>
+<contactref element="C22" pad="2"/>
+<contactref element="C23" pad="2"/>
+<contactref element="C24" pad="2"/>
 <wire x1="-47.991" y1="-197.104" x2="-50.978" y2="-197.997" width="0" layer="19" extent="1-1"/>
 <wire x1="-54.872" y1="-203.538" x2="-50.978" y2="-197.997" width="0" layer="19" extent="1-1"/>
@@
 <wire x1="-75.112" y1="-244.856" x2="-76.272" y2="-241.554" width="0" layer="19" extent="1-1"/>
 <wire x1="-76.272" y1="-260.096" x2="-75.112" y2="-244.856" width="0" layer="19" extent="1-1"/>
+<wire x1="-75.192" y1="-263.144" x2="-76.272" y2="-260.096" width="0" layer="19" extent="1-1"/>
+<wire x1="-75.192" y1="-266.192" x2="-75.192" y2="-263.144" width="0" layer="19" extent="1-1"/>
+<wire x1="-75.192" y1="-276.86" x2="-75.192" y2="-266.192" width="0" layer="19" extent="1-1"/>
+<wire x1="-75.112" y1="-282.956" x2="-75.192" y2="-276.86" width="0" layer="19" extent="1-1"/>
 <wire x1="-16.903" y1="-171.45" x2="-39.869" y2="-197.836" width="0" layer="19" extent="1-1"/>
 <wire x1="-17.708" y1="-157.48" x2="-16.903" y2="-171.45" width="0" layer="19" extent="1-1"/>
@@
 <contactref element="U6" pad="12"/>
 <contactref element="U6" pad="1"/>
+<contactref element="U4" pad="1"/>
+<contactref element="U4" pad="10"/>
+<contactref element="C21" pad="1"/>
+<contactref element="C22" pad="1"/>
 <wire x1="-54.022" y1="-203.188" x2="-35.462" y2="-198.374" width="0" layer="19" extent="1-1"/>
 <wire x1="-55.872" y1="-203.538" x2="-54.022" y2="-203.188" width="0" layer="19" extent="1-1"/>
@@
 <wire x1="-54.872" y1="-201.338" x2="-56.722" y2="-201.688" width="0" layer="19" extent="1-1"/>
 <wire x1="-56.888" y1="-205.74" x2="-55.872" y2="-203.538" width="0" layer="19" extent="1-1"/>
+<wire x1="-59.56" y1="-202.962" x2="-56.722" y2="-201.688" width="0" layer="19" extent="1-1"/>
+<wire x1="-62.36" y1="-202.962" x2="-59.56" y2="-202.962" width="0" layer="19" extent="1-1"/>
 <wire x1="-18.868" y1="-157.48" x2="-35.462" y2="-198.374" width="0" layer="19" extent="1-1"/>
 <wire x1="-12.132" y1="-150.126" x2="-18.868" y2="-157.48" width="0" layer="19" extent="1-1"/>
@@
 <wire x1="33.556" y1="14.981" x2="23.3506" y2="12.7254" width="0" layer="19" extent="1-1"/>
 <wire x1="34.2434" y1="20.574" x2="34.798" y2="14.986" width="0" layer="19" extent="1-1"/>
+<wire x1="-76.192" y1="-263.144" x2="-56.888" y2="-205.74" width="0" layer="19" extent="1-1"/>
+<wire x1="-76.192" y1="-266.192" x2="-76.192" y2="-263.144" width="0" layer="19" extent="1-1"/>
 </signal>
 <signal name="!RESET">
@@
 <signal name="VIN">
 <contactref element="U8" pad="7"/>
+<contactref element="U4" pad="5"/>
+<contactref element="C23" pad="1"/>
+<contactref element="R21" pad="2"/>
+<wire x1="-76.192" y1="-276.86" x2="-75.192" y2="-279.908" width="0" layer="19" extent="1-1"/>
+<wire x1="-61.392" y1="-210.241" x2="-76.192" y2="-276.86" width="0" layer="19" extent="1-1"/>
+<wire x1="-62.36" y1="-204.962" x2="-61.392" y2="-210.241" width="0" layer="19" extent="1-1"/>
 </signal>
 <signal name="N$9">
@@
 <wire x1="-65.113" y1="-204.962" x2="-75.112" y2="-260.096" width="0" layer="19" extent="1-1"/>
 </signal>
+<signal name="N$20">
+<contactref element="U4" pad="4"/>
+<contactref element="L3" pad="2"/>
+<wire x1="-62.36" y1="-204.462" x2="-73.068" y2="-271.526" width="0" layer="19" extent="1-1"/>
+</signal>
+<signal name="N$21">
+<contactref element="U4" pad="2"/>
+<contactref element="L3" pad="1"/>
+<wire x1="-62.36" y1="-203.462" x2="-75.268" y2="-271.526" width="0" layer="19" extent="1-1"/>
+</signal>
+<signal name="N$22">
+<contactref element="C24" pad="1"/>
+<contactref element="R21" pad="1"/>
+<contactref element="U4" pad="8"/>
+<contactref element="U4" pad="7"/>
+<contactref element="U4" pad="6"/>
+<wire x1="-76.192" y1="-279.908" x2="-76.272" y2="-282.956" width="0" layer="19" extent="1-1"/>
+<wire x1="-59.56" y1="-204.962" x2="-76.192" y2="-279.908" width="0" layer="19" extent="1-1"/>
+<wire x1="-59.56" y1="-204.462" x2="-59.56" y2="-204.962" width="0" layer="19" extent="1-1"/>
+<wire x1="-59.56" y1="-203.962" x2="-59.56" y2="-204.462" width="0" layer="19" extent="1-1"/>
+</signal>
 </signals>
