File: pi_day_2025.brd (EAGLE design)
At the start: 50.8 x 25.4 mm, 109 parts, among them IC1 W25Q64JVXGIQ, J4 SM03B-SRSS-TB(LF)(SN), Q2 310mA/60V/1.6Ω, U1 APS6404L-3SQR-ZR, U2 RP2350A, U3 TPS76318DBVRG4, U4 TPS63001DRCR, U5 TXS0108EPWRG4, U6 LSM6DS3TR-C, U7 MCP73833T-AMI/MF, U8 TPS2113APWR, U9 ESP32-C3-MINI-1-N4, Y1 12MHz

Commit message: Finished schematic
Parts:
- removed C1: 0.1uF, SparkFun-Capacitors:0402-TIGHT
- removed C10, C11, C48, C8, C9: 0.1uF, SparkFun-Capacitors:0402
- removed C47: 10uF, SparkFun-Capacitors:0402-TIGHT
- removed D10, D7, D8, D9: SK6812-EJ, SK6812-E:LED_SK6812-E
- removed R1, R23: 10k, SparkFun-Resistors:0402
- removed U1: APS6404L-3SQR-ZR, RP2350A:APS6404L-3SQR-ZR
- removed U9: ESP32-C3-MINI-1-N4, ESP32-C3-MINI-1-N4:XCVR_ESP32-C3-MINI-1-N4
- moved U2 130.4 mm to (-103.4, -39.3), turned to 180 degrees
- moved D6 112.6 mm to (-0.71, 8.12), turned to 90 degrees
- moved C12 108.7 mm to (-96.2, -9.45)
- moved D4 108.6 mm to (26.1, 17.3), turned to 270 degrees
- moved C17 108.2 mm to (-98.7, -23.6)
- moved C18 108.2 mm to (-90.4, -24.4)
- moved C27 108.2 mm to (-86.2, -26.0)
- moved C28 108.2 mm to (-79.1, -20.6)
- moved C29 108.2 mm to (-86.7, -13.5)
- moved C30 108.2 mm to (-83.7, -14.6)
- moved C32 108.2 mm to (-89.1, -13.4)
- moved C34 108.2 mm to (-90.0, -13.4)
- moved C36 108.2 mm to (-98.2, -17.5)
- moved C37 108.2 mm to (-94.6, -17.3)
- moved C38 108.2 mm to (-87.7, -13.5)
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Connections:
- removed net !ESP32_BOOT: U2.31, U9.23
- removed net !ESP32_RST: U2.29, U9.8
- removed net !FLASH_CS: R1.2, U1.1, U2.2
- removed net ESP32_CS: U2.33, U9.16
- removed net ESP32_HANDSHAKE: U2.28, U9.6
- removed net ESP32_MISO: U2.32, U9.5
- removed net ESP32_MOSI: U2.35, U9.21
- removed net ESP32_RX: U2.16, U9.30
- removed net ESP32_SCK: U2.34, U9.20
- removed net ESP32_TX: U2.17, U9.31
- removed net N$25: R23.1, U9.22
- removed net NPXL_6_OUT: D6.2, D7.4
- removed net NPXL_7_OUT: D7.2, D8.4
- removed net NPXL_8_OUT: D8.2, D9.4
- removed net NPXL_9_OUT: D10.4, D9.2
- net 3.3V: no longer C1.1, C10.1, C11.1, C47.1, C48.1, C8.1, C9.1, D10.1, D7.1, D8.1, D9.1, R1.1, R23.2, U1.8, U9.3
- net GND: no longer C1.2, C10.2, C11.2, C47.2, C48.2, C8.2, C9.2, D10.3, D7.3, D8.3, D9.3, U1.4, U1.9, U9.1, U9.11, U9.14, U9.2, U9.36, U9.37, U9.38, U9.39, U9.40, U9.41, U9.42, U9.43, U9.44, U9.45, U9.46, U9.47, U9.48, U9.49_1, U9.49_2, U9.49_3, U9.49_4, U9.49_5, U9.49_6, U9.49_7, U9.49_8, U9.49_9, U9.50, U9.51, U9.52, U9.53
- net QSPI_CLK: no longer U1.6
- net SIO0: no longer U1.5
- net SIO1: no longer U1.2
- net SIO2: no longer U1.3
- net SIO3: no longer U1.7
Routing:
- net SCL: track 59.7 -> 0.00 mm, vias 3 -> 0
- net SDA: track 56.6 -> 0.00 mm, vias 2 -> 0
- net 3.3V: track 52.9 -> 0.00 mm, vias 14 -> 0
- net 1.1V: track 46.3 -> 0.00 mm, vias 4 -> 0
- net N$27: track 24.9 -> 0.00 mm, vias 2 -> 0
- net SIO1: track 20.5 -> 0.00 mm, vias 2 -> 0
- net SIO2: track 19.2 -> 0.00 mm, vias 2 -> 0
- net VBUS: track 19.0 -> 0.00 mm, vias 2 -> 0
- net !QSPI_CS: track 17.2 -> 0.00 mm
- net SIO3: track 16.2 -> 0.00 mm, vias 2 -> 0
- net USB_N: track 15.7 -> 0.00 mm
- net QSPI_CLK: track 15.7 -> 0.00 mm, vias 2 -> 0
- net !RESET: track 14.4 -> 0.00 mm, vias 2 -> 0
- net SIO0: track 14.3 -> 0.00 mm, vias 2 -> 0
- net !BOOT: track 12.9 -> 0.00 mm, vias 2 -> 0
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- removed copper zone on layer 15, net 3.3V
- removed copper zone on layer 1, net GND
- removed copper zone on layer 16, net GND
- removed copper zone on layer 2, net GND
Other:
- board size 50.8 x 25.4 mm -> 70 x 79.5 mm
