File: pi_day_2025.brd (EAGLE design)
At the start: 70 x 79.5 mm, 99 parts, among them IC1 W25Q64JVXGIQ, IC2 NPM1300-QEAA-R, J4 SM03B-SRSS-TB(LF)(SN), Q2 310mA/60V/1.6Ω, U1 APS6404L-3SQR-ZR, U2 RP2350A, U5 TXS0108EPWRG4, U6 LSM6DS3TR-C, U9 ESP32-C3-MINI-1-N4, Y1 12MHz

Commit message: Checkin
Parts:
- removed R8: 0, SparkFun-Resistors_Sai:0402
- added 1.8V, 3.3V, GND, VBATT, VBUS, VSYS, V_USB_OUT: TPB1,27, testpad:B1,27
- added C25: 10uF, SparkFun-Capacitors_Sai:0402
- added C26, C51: 0.1uF, SparkFun-Capacitors_Sai:0402
- added C49, C50, C52: 0.1uF, SparkFun-Capacitors:0402
- added J2: Qwiic, SparkFun-Connectors:1X04_1MM_RA
- added S4: MOMENTARY-SWITCH-SPST-SMD-4.6X2.8MM, SparkFun-Switches:TACTILE_SWITCH_SMD_4.6X2.8MM
- added U15: SN74LVC1T45DBVRG4, SN74LVC1T45DBVRG4:SOT95P280X145-6N
- added U3: XTSD04GLGEAG, XTSD04GLGEAG:SON127P600X800X95-8N
- C1, C18, C19, C27, C28, C29, C30, C31, C32, C33, C34, C35, C36, C37, C38, C39, C40: device SparkFun-Capacitors:0402-TIGHT -> SparkFun-Capacitors_Sai:0402
- C17: device SparkFun-Capacitors:0402 -> SparkFun-Capacitors_Sai:0402
- J1: value (none) -> JST-PH=2
- L2: value 3.3µH -> 3.3uH; device SparkFun-Coils:0805 -> LQH2MCN120K02L:IND_LQH2MCN120K02L
- LS1: device CSS-0575A-SMT:CUI_CSS-0575A-SMT -> CMT-8504-100-SMT-TR:XDCR_CMT-8504-100-SMT-TR
- Q2: value 310mA/60V/1.6Ω -> BSS138; device SparkFun-DiscreteSemi:SOT323 -> BSS138:SOT95P240X111-3N
- R10: value (none) -> 470K
- R12, R13: device SparkFun-Resistors:0402-TIGHT -> SparkFun-Resistors_Sai:0402
- R2: value 100 -> 100OHM; device SparkFun-Resistors:0402-TIGHT -> SparkFun-Resistors_Sai:0402
- R4: value (none) -> DNF
- R5: value (none) -> 1K
- R6, R7: value (none) -> 2.2K
- R9: value 47KOHM-0402-1/10W-10% -> 47K
- moved C24 195.0 mm to (-15.6, 9.96), turned to 180 degrees
- moved L4 192.8 mm to (-21.8, 8.05), turned to 180 degrees
- moved R16 189.6 mm to (-17.6, 12.0), turned to 270 degrees
- moved L3 189.0 mm to (-17.5, 8.08)
- moved R14 184.3 mm to (-22.0, 11.9), turned to 270 degrees
- moved C23 174.0 mm to (-18.1, 9.96)
- moved LED1 172.8 mm to (-12.4, 1.04), turned to 180 degrees
- moved C22 169.2 mm to (-21.4, 9.96), turned to 180 degrees
- moved R22 159.7 mm to (22.4, 6.20), turned to 270 degrees
- moved C21 156.5 mm to (-18.5, -4.95), turned to 270 degrees
- moved C20 152.9 mm to (-20.3, -4.95), turned to 270 degrees
- moved C44 152.6 mm to (25.6, -2.34), turned to 270 degrees
- moved C43 149.9 mm to (24.2, -2.34), turned to 270 degrees
- moved C45 148.3 mm to (18.7, -2.36), turned to 90 degrees
- moved C16 146.1 mm to (-24.9, 3.12)
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Connections:
- removed net CHARGE_STAT: U2.3
- removed net LSIN1/VINLDO1: IC2.28
- removed net LSIN2/VINLDO2: IC2.30
- removed net LSOUT1/VOUTLDO1: IC2.29
- removed net LSOUT2/VOUTLDO2: IC2.31
- removed net N$38: J1.2
- removed net N$8: IC2.15, R8.2
- new net !MEM_CS: U2.13, U3.2
- new net !RESET_NPM1300: IC2.7, S4.3, S4.4
- new net NPXL_3.3V: U15.3, U2.40
- new net V_USB_OUT: C15.1, IC2.22, V_USB_OUT.TP
- net !INT_NPM1300: now also U2.42; no longer U2.10
- net 1.1V: now also L2.1; no longer L2.2
- net 1.8V: now also 1.8V.TP
- net 3.3V: now also 3.3V.TP, C25.1, C26.1, C49.2, C51.2, C52.1, J2.2, LS1.P, U15.1, U15.5, U3.8; no longer C10.1, C11.1, C2.1, C3.1, C4.1, C5.1, C6.1, C7.1, C8.1, C9.1, D1.1, D10.1, D2.1, D3.1, D4.1, D5.1, D6.1, D7.1, D8.1, D9.1, LS1.1
- net ESP32_MISO: now also U3.6
- net ESP32_MOSI: now also U3.5
- net ESP32_SCK: now also U3.3
- net GND: now also C26.2, C49.1, C50.2, C51.1, C52.2, GND.TP, IC2.28, IC2.29, IC2.30, IC2.31, J2.1, S4.1, S4.2, U15.2, U3.4; no longer R8.1
- net N$26: now also LS1.N; no longer LS1.2
- net N$5: now also L2.2; no longer L2.1
- net N$9: now also J1.2
- net NPXL_1_IN: now also U15.4; no longer U2.13
- net PVSS2: now also C25.2
- net SCL: now also J2.4
- net SDA: now also J2.3
- net USB_CC1: now also CONN1.A5
- net VSYS: now also C10.1, C11.1, C2.1, C3.1, C4.1, C5.1, C50.1, C6.1, C7.1, C8.1, C9.1, D1.1, D10.1, D2.1, D3.1, D4.1, D5.1, D6.1, D7.1, D8.1, D9.1, U15.6, VSYS.TP
- net V_BATT: now also VBATT.TP
- net V_USB: now also VBUS.TP; no longer C15.1, IC2.22
Routing:
- net SDA: track 0.00 -> 135.5 mm, vias 0 -> 4
- net 3.3V: track 0.00 -> 134.4 mm, vias 0 -> 28
- net SCL: track 0.00 -> 133.2 mm, vias 0 -> 2
- net VSYS: track 0.00 -> 128.7 mm, vias 0 -> 14
- net NPXL_9_OUT: track 0.00 -> 78.6 mm, vias 0 -> 3
- net ESP32_HANDSHAKE: track 0.00 -> 74.2 mm, vias 0 -> 2
- net ESP32_MISO: track 0.00 -> 65.7 mm, vias 0 -> 2
- net 1.8V: track 0.00 -> 64.4 mm, vias 0 -> 2
- net ESP32_MOSI: track 0.00 -> 64.3 mm
- net LSM6_INT1: track 0.00 -> 62.5 mm, vias 0 -> 2
- net ESP32_SCK: track 0.00 -> 62.3 mm, vias 0 -> 2
- net BUZZER_DRIVER: track 0.00 -> 61.0 mm, vias 0 -> 2
- net ESP32_CS: track 0.00 -> 58.7 mm, vias 0 -> 2
- net !ESP32_BOOT: track 0.00 -> 55.9 mm
- net !ESP32_RST: track 0.00 -> 55.7 mm, vias 0 -> 2
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- added copper zone on layer 15, net 3.3V
- added copper zone on layer 1, net GND
- added copper zone on layer 16, net GND
- added copper zone on layer 2, net GND
- added copper zone on layer 15, net VSYS
Other:
- board text removed: "GND"
